File: Tesla_Coil/MMS_SSTC/PSU.kicad_sch (KiCad schematic)
At the start: 15 parts, among them J2 Screw_Terminal_01x02, SW1 SW_SPST, U4 LM7812_TO220

Commit message: Rough layout on final SSTC PCB
Other:
- note removed: "adding an ICL is pointless unless we design the circuit such that the logic turns off immediately so the FET doesn't drain the caps. You could just cycle it on and off and render the ICL useless because it would still be hot but the caps are drained so just use a slightly better rectifier"
Changed lines of the file:
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@@
-		)
-	)
-	(text "adding an ICL is pointless unless we design the circuit\nsuch that the logic turns off immediately so the FET doesn't\ndrain the caps. You could just cycle it on and off and render\nthe ICL useless because it would still be hot but the caps are drained\nso just use a slightly better rectifier"
-		(exclude_from_sim no)
-		(at 217.424 31.242 0)
-		(effects
-			(font
-				(size 1.27 1.27)
-			)
 		)
 	)

Commit message: route SSTC PCB and then find out critical problem yay
Parts:
- renumbered D7 to LED1
Changed lines of the file:
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@@
 		(on_board yes)
 		(dnp no)
-		(fields_autoplaced yes)
-		(property "Reference" "D7"
-			(at 83.82 131.1274 90)
+		(property "Reference" "LED1"
+			(at 82.55 130.81 90)
 			(effects
 				(font
@@
 				)
 				(justify right)
+				(hide yes)
 			)
 		)
@@
 			(project ""
 				(path "/b29a3901-c128-4c19-b69f-61de71283b43/bfaa6adf-6b83-46d0-b8b3-f415df3d6008"
-					(reference "D7")
+					(reference "LED1")
 					(unit 1)
 				)

Commit message: FINISH THE DAMN THING
Parts:
- added C13, C14: 0.1u, Capacitor_THT:C_Disc_D3.0mm_W2.0mm_P2.50mm, symbol Device:C_Small
- added U5: LM7805_TO220, Package_TO_SOT_THT:TO-220-3_Vertical, symbol Regulator_Linear:LM7805_TO220
Connections:
- net +12V: now also C13.1, U5.1 (VI)
- net GND: now also C13.2, C14.2, U5.2 (GND)
- new net +5V: C14.1, U5.3 (VO)
